File: SIOM/KiCad/ValveCtrl.sch (KiCad schematic (older format))
At the start: 10 parts, among them U601 LM7332

Commit message: KiCad files SIOM_def
Parts:
- added C502: 10uF 50V, Capacitor_SMD:CP_Elec_5x5.3, symbol Device:CP
- C501: renamed from C601; value 100n/16 -> 100nF 50V
- R501: renamed from R603; value 22k0 -> 10K
- R502: renamed from R606; value 22k0 -> 10K
- R503: renamed from R602; value 10k0 -> 22K
- R504: renamed from R605; value 10k0 -> 22K
- renumbered D601 to D501, D602 to D502, R601 to R505, R604 to R506, U601 to U501
Connections:
- net +12V: now also C502.1
- net GND: now also C502.2
- net ANA_OUT_01 renamed DAC1_OUT1_VALVE_1
- net ANA_OUT_02 renamed DAC1_OUT2_VALVE_2
Changed lines of the file:
@@
 EESchema Schematic File Version 4
-LIBS:SIOMv01-cache
 EELAYER 30 0
 EELAYER END
 $Descr A4 11693 8268
 encoding utf-8
-Sheet 6 9
+Sheet 5 10
 Title ""
 Date ""
@@
 $EndDescr
 $Comp
-L Amplifier_Operational:LM7332 U601
+L Amplifier_Operational:LM7332 U501
 U 1 1 5FA46782
 P 5500 2100
-F 0 "U601" H 5550 2400 50  0000 C CNN
+F 0 "U501" H 5550 2400 50  0000 C CNN
 F 1 "LM7332" H 5550 2300 50  0000 C CNN
 F 2 "Package_SO:SOIC-8_3.9x4.9mm_P1.27mm" H 5450 2200 50  0001 C CNN
@@
 	5150 2200 5150 2400
 $Comp
-L SIOMv01-rescue:R-Device R602
+L SIOMv01-rescue:R-Device R503
 U 1 1 5FA48E11
 P 5500 2400
-F 0 "R602" V 5400 2400 50  0000 C CNN
-F 1 "10k0" V 5500 2400 50  0000 C CNN
+F 0 "R503" V 5400 2400 50  0000 C CNN
+F 1 "22K" V 5600 2400 50  0000 C CNN
 F 2 "Resistor_SMD:R_0603_1608Metric" V 5430 2400 50  0001 C CNN
 F 3 "~" H 5500 2400 50  0001 C CNN
@@
 Connection ~ 5150 2400
 $Comp
-L SIOMv01-rescue:R-Device R603
+L SIOMv01-rescue:R-Device R501
 U 1 1 5FA49C27
 P 5150 2600
-F 0 "R603" H 5200 2600 50  0000 L CNN
-F 1 "22k0" V 5150 2500 50  0000 L CNN
+F 0 "R501" H 5200 2600 50  0000 L CNN
+F 1 "10K" H 5250 2500 50  0000 L CNN
 F 2 "Resistor_SMD:R_0603_1608Metric" V 5080 2600 50  0001 C CNN
 F 3 "~" H 5150 2600 50  0001 C CNN
@@
 $EndComp
 $Comp
-L SIOMv01-rescue:GND-power #PWR0601
+L SIOMv01-rescue:GND-power #PWR0501
 U 1 1 5FA4A713
 P 5150 2800
-F 0 "#PWR0601" H 5150 2550 50  0001 C CNN
+F 0 "#PWR0501" H 5150 2550 50  0001 C CNN
 F 1 "GND" H 5155 2627 50  0000 C CNN
 F 2 "" H 5150 2800 50  0001 C CNN
@@
 	5150 2800 5150 2750
 $Comp
-L Amplifier_Operational:LM7332 U601
+L Amplifier_Operational:LM7332 U501
 U 2 1 5FA507BC
 P 5500 3450
-F 0 "U601" H 5550 3750 50  0000 C CNN
+F 0 "U501" H 5550 3750 50  0000 C CNN
 F 1 "LM7332" H 5550 3650 50  0000 C CNN
 F 2 "Package_SO:SOIC-8_3.9x4.9mm_P1.27mm" H 5450 3550 50  0001 C CNN
@@
 	5150 3550 5150 3750
 $Comp
-L SIOMv01-rescue:R-Device R605
+L SIOMv01-rescue:R-Device R504
 U 1 1 5FA507C6
 P 5500 3750
-F 0 "R605" V 5400 3750 50  0000 C CNN
-F 1 "10k0" V 5500 3750 50  0000 C CNN
+F 0 "R504" V 5400 3750 50  0000 C CNN
+F 1 "22K" V 5600 3750 50  0000 C CNN
 F 2 "Resistor_SMD:R_0603_1608Metric" V 5430 3750 50  0001 C CNN
 F 3 "~" H 5500 3750 50  0001 C CNN
@@
 Connection ~ 5150 3750
 $Comp
-L SIOMv01-rescue:R-Device R606
+L SIOMv01-rescue:R-Device R502
 U 1 1 5FA507D3
 P 5150 3950
-F 0 "R606" H 5200 3950 50  0000 L CNN
-F 1 "22k0" V 5150 3850 50  0000 L CNN
+F 0 "R502" H 5200 3950 50  0000 L CNN
+F 1 "10K" H 5200 3850 50  0000 L CNN
 F 2 "Resistor_SMD:R_0603_1608Metric" V 5080 3950 50  0001 C CNN
 F 3 "~" H 5150 3950 50  0001 C CNN
@@
 $EndComp
 $Comp
-L SIOMv01-rescue:GND-power #PWR0603
+L SIOMv01-rescue:GND-power #PWR0502
 U 1 1 5FA507D9
 P 5150 4150
-F 0 "#PWR0603" H 5150 3900 50  0001 C CNN
+F 0 "#PWR0502" H 5150 3900 50  0001 C CNN
 F 1 "GND" H 5155 3977 50  0000 C CNN
 F 2 "" H 5150 4150 50  0001 C CNN
@@
 	5150 4150 5150 4100
 $Comp
-L Amplifier_Operational:LM7332 U601
+L Amplifier_Operational:LM7332 U501
 U 3 1 5FA56DF7
 P 5450 5200
-F 0 "U601" H 5408 5246 50  0000 L CNN
+F 0 "U501" H 5408 5246 50  0000 L CNN
 F 1 "LM7332" H 5408 5155 50  0000 L CNN
 F 2 "Package_SO:SOIC-8_3.9x4.9mm_P1.27mm" H 5400 5300 50  0001 C CNN
@@
 $EndComp
 $Comp
-L SIOMv01-rescue:GND-power #PWR0606
+L SIOMv01-rescue:GND-power #PWR0504
 U 1 1 5FA5D9F0
 P 5350 5600
-F 0 "#PWR0606" H 5350 5350 50  0001 C CNN
+F 0 "#PWR0504" H 5350 5350 50  0001 C CNN
 F 1 "GND" H 5355 5427 50  0000 C CNN
 F 2 "" H 5350 5600 50  0001 C CNN
@@
 	5350 4800 5350 4850
 $Comp
-L SIOMv01-rescue:+12V-power #PWR0605
+L SIOMv01-rescue:+12V-power #PWR0503
 U 1 1 5FA60B81
 P 5350 4800
-F 0 "#PWR0605" H 5350 4650 50  0001 C CNN
+F 0 "#PWR0503" H 5350 4650 50  0001 C CNN
 F 1 "+12V" H 5365 4973 50  0000 C CNN
 F 2 "" H 5350 4800 50  0001 C CNN
@@
 $EndComp
 $Comp
-L SIOMv01-rescue:C-Device C601
+L SIOMv01-rescue:C-Device C501
 U 1 1 5FA626C1
 P 5800 5200
-F 0 "C601" H 5915 5246 50  0000 L CNN
-F 1 "100n/16" H 5915 5155 50  0000 L CNN
+F 0 "C501" H 5915 5246 50  0000 L CNN
+F 1 "100nF 50V" H 5915 5155 50  0000 L CNN
 F 2 "Capacitor_SMD:C_0603_1608Metric" H 5838 5050 50  0001 C CNN
 F 3 "~" H 5800 5200 50  0001 C CNN
@@
 	5350 5550 5350 5500
 $Comp
-L SIOMv01-rescue:R-Device R601
+L SIOMv01-rescue:R-Device R505
 U 1 1 5FA72B27
 P 6150 2100
-F 0 "R601" V 6050 2100 50  0000 C CNN
-F 1 "470R" V 6150 2100 50  0000 C CNN
+F 0 "R505" V 6050 2100 50  0000 C CNN
+F 1 "470R" V 6250 2100 50  0000 C CNN
 F 2 "Resistor_SMD:R_0603_1608Metric" V 6080 2100 50  0001 C CNN
 F 3 "~" H 6150 2100 50  0001 C CNN
@@
 $EndComp
 $Comp
-L SIOMv01-rescue:R-Device R604
+L SIOMv01-rescue:R-Device R506
 U 1 1 5FA8B859
 P 6150 3450
-F 0 "R604" V 6050 3450 50  0000 C CNN
-F 1 "470R" V 6150 3450 50  0000 C CNN
+F 0 "R506" V 6050 3450 50  0000 C CNN
+F 1 "470R" V 6250 3450 50  0000 C CNN
 F 2 "Resistor_SMD:R_0603_1608Metric" V 6080 3450 50  0001 C CNN
 F 3 "~" H 6150 3450 50  0001 C CNN
@@
 $EndComp
 $Comp
-L SIOMv01-rescue:DZ2S120X0L-Diode D601
+L SIOMv01-rescue:DZ2S120X0L-Diode D501
 U 1 1 5FA8ED42
 P 5950 2600
-F 0 "D601" V 5904 2680 50  0000 L CNN
+F 0 "D501" V 5904 2680 50  0000 L CNN
 F 1 "DZ2S120X0L" V 5995 2680 50  0000 L CNN
 F 2 "Diode_SMD:D_SOD-523" H 5950 2425 50  0001 C CNN
@@
 $EndComp
 $Comp
-L SIOMv01-rescue:GND-power #PWR0602
+L SIOMv01-rescue:GND-power #PWR0505
 U 1 1 5FAA36F5
 P 5950 2800
-F 0 "#PWR0602" H 5950 2550 50  0001 C CNN
+F 0 "#PWR0505" H 5950 2550 50  0001 C CNN
 F 1 "GND" H 5955 2627 50  0000 C CNN
 F 2 "" H 5950 2800 50  0001 C CNN
@@
 	5950 2100 6000 2100
 $Comp
-L SIOMv01-rescue:DZ2S120X0L-Diode D602
+L SIOMv01-rescue:DZ2S120X0L-Diode D502
 U 1 1 5FAAA996
 P 5950 3950
-F 0 "D602" V 5904 4030 50  0000 L CNN
+F 0 "D502" V 5904 4030 50  0000 L CNN
 F 1 "DZ2S120X0L" V 5995 4030 50  0000 L CNN
 F 2 "Diode_SMD:D_SOD-523" H 5950 3775 50  0001 C CNN
@@
 $EndComp
 $Comp
-L SIOMv01-rescue:GND-power #PWR0604
+L SIOMv01-rescue:GND-power #PWR0506
 U 1 1 5FAAA99C
 P 5950 4150
-F 0 "#PWR0604" H 5950 3900 50  0001 C CNN
+F 0 "#PWR0506" H 5950 3900 50  0001 C CNN
 F 1 "GND" H 5955 3977 50  0000 C CNN
 F 2 "" H 5950 4150 50  0001 C CNN
@@
 Text Notes 5900 5400 0    50   ~ 0
 Near IC
-Text Label 4600 3350 0    50   ~ 0
-ANA_OUT_02
-Text Label 4600 2000 0    50   ~ 0
-ANA_OUT_01
 Wire Wire Line
 	4550 3350 5200 3350
@@
 	4550 2000 5200 2000
 Text HLabel 4550 2000 0    50   Input ~ 0
-ANA_OUT_01
+DAC1_OUT1_VALVE_1
 Text HLabel 4550 3350 0    50   Input ~ 0
-ANA_OUT_02
+DAC1_OUT2_VALVE_2
+$Comp
+L Device:CP C502
+U 1 1 6090E3EF
+P 4800 5200
+F 0 "C502" H 4918 5246 50  0000 L CNN
+F 1 "10uF 50V" H 4918 5155 50  0000 L CNN
+F 2 "Capacitor_SMD:CP_Elec_5x5.3" H 4838 5050 50  0001 C CNN
+F 3 "~" H 4800 5200 50  0001 C CNN
+	1    4800 5200
+	1    0    0    -1
+$EndComp
+Wire Wire Line
+	4800 5350 4800 5550
+Wire Wire Line
+	4800 5050 4800 4850
+Wire Wire Line
+	4800 4850 5350 4850
+Wire Wire Line
+	4800 5550 5350 5550
 $EndSCHEMATC
